File: aux_circuit.kicad_sch (KiCad schematic)
At the start: 23 parts, among them IC2 LM5169PQDDARQ1, U1 MGJ2D151505SC, U2 MGJ2D151505SC, U4 3.3V reg

Commit message: V1
layout and tracing done
Parts:
- added JP1, JP2: jumper, Jumper:SolderJumper-2_P1.3mm_Open_RoundedPad1.0x1.5mm, symbol Jumper:SolderJumper_2_Bridged
- renumbered D3 to D8, R1 to R13, R9 to R15, R1 to RT1, R1 to Rf1, R1 to Rf2, R1 to Rsnub1, TP1 to TP6, TP1 to TP7
Connections:
- net +15V: now also JP2.1 (A); no longer TP6.1, U1.1 (+VIN), U2.1 (+VIN), U4.2 (IN)
- net 100V: now also JP1.1 (A); no longer Cin1.1, IC2.2 (VIN), IC2.3 (EN/UVLO)
- new net: JP2.2 (B), TP6.1, U1.1 (+VIN), U2.1 (+VIN), U4.2 (IN)
- new net: Cin1.1, IC2.2 (VIN), IC2.3 (EN/UVLO), JP1.2 (B)
Other:
- moved on the sheet: C10, C11, C9, Cbst1, Cin1, Cout1, Cout2, Cout3, Csnub1, D8, IC2, L2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
