File: gatedriver.kicad_sch (KiCad schematic)
At the start: 26 parts, among them IC1 2EDF7275FXUMA2, J4 RP2040 connector

Commit message: V1
layout and tracing done
Parts:
- renumbered R2 to R1, R2 to R5, R2 to R6
Connections:
- net PWM1: now also J4.3 (Pin_3); no longer J4.2 (Pin_2)
- net PWM2: now also J4.2 (Pin_2); no longer J4.3 (Pin_3)
Other:
- moved on the sheet: J4
