File: power.kicad_sch (KiCad schematic)
At the start: 18 parts, among them J1 Conn_01x02_Socket, J2 output, Q1 IPP50R280CE, Q2 IPP50R280CE

Commit message: V1
layout and tracing done
Parts:
- removed TP5: Vout, 5001 tp:KEYSTONE_5001, symbol Connector:TestPoint
- added H1, H2, H3, H4: MountingHole, MountingHole:MountingHole_3.2mm_M3, symbol Mechanical:MountingHole
- renumbered C1 to C2, C1 to C3, C1 to C4, R1 to R3, R2 to R4, R1 to R7, R1 to R8
Connections:
- net 100V: now also Q1.2 (D); no longer Q1.1 (D)
- net GND: now also J2.1 (Pin_1); no longer J2.2 (Pin_2)
- net Gate1: now also Q1.1 (G); no longer Q1.2 (G)
- net Gate2: now also Q2.1 (G); no longer Q2.2 (G)
- net iso1-0V: now also Q2.2 (D); no longer Q2.1 (D)
- net at C1.1, C2.1, C3.1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: now also J2.2 (Pin_2); no longer J2.1 (Pin_1)

Commit message: Full design files with codes
Parts:
- Q1, Q2: value IPP50R280CE -> IGLD60R190D1
Other:
- moved on the sheet: H1, H2, H3, H4, J1
Changed lines of the file:
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@@
 	(wire
 		(pts
-			(xy 39.37 104.14) (xy 39.37 100.33)
+			(xy 77.47 95.25) (xy 77.47 91.44)
 		)
 		(stroke
@@
 	(wire
 		(pts
-			(xy 41.91 97.79) (xy 39.37 97.79)
+			(xy 80.01 88.9) (xy 77.47 88.9)
 		)
 		(stroke
@@
 	(global_label "100V"
 		(shape input)
-		(at 41.91 97.79 0)
+		(at 80.01 88.9 0)
 		(fields_autoplaced yes)
 		(effects
@@
 		)
 		(property "Intersheetrefs" "${INTERSHEET_REFS}"
-			(at 47.3542 97.79 0)
+			(at 85.4542 88.9 0)
 			(effects
 				(font
@@
 	(symbol
 		(lib_id "Mechanical:MountingHole")
-		(at 69.85 171.45 0)
+		(at 90.17 114.3 0)
 		(unit 1)
 		(exclude_from_sim no)
@@
 		(fields_autoplaced yes)
 		(property "Reference" "H2"
-			(at 72.39 170.1799 0)
+			(at 92.71 113.0299 0)
 			(effects
 				(font
@@
 		)
 		(property "Value" "MountingHole"
-			(at 72.39 172.7199 0)
+			(at 92.71 115.5699 0)
 			(effects
 				(font
@@
 		)
 		(property "Footprint" "MountingHole:MountingHole_3.2mm_M3"
-			(at 69.85 171.45 0)
+			(at 90.17 114.3 0)
 			(effects
 				(font
@@
 		)
 		(property "Datasheet" "~"
-			(at 69.85 171.45 0)
+			(at 90.17 114.3 0)
 			(effects
 				(font
@@
 		)
 		(property "Description" "Mounting Hole without connection"
-			(at 69.85 171.45 0)
+			(at 90.17 114.3 0)
 			(effects
 				(font
@@
 		(fields_autoplaced yes)
 		(property "Reference" "Q1"
-			(at 128.27 74.93 0)
-			(effects
-				(font
-					(size 1.27 1.27)
-				)
-				(justify left)
-			)
-		)
-		(property "Value" "IPP50R280CE"
-			(at 128.27 77.47 0)
+			(at 128.27 74.9299 0)
+			(effects
+				(font
+					(size 1.27 1.27)
+				)
+				(justify left)
+			)
+		)
+		(property "Value" "IGLD60R190D1"
+			(at 128.27 77.4699 0)
 			(effects
 				(font
@@
 	(symbol
 		(lib_id "Mechanical:MountingHole")
-		(at 46.99 171.45 0)
+		(at 67.31 114.3 0)
 		(unit 1)
 		(exclude_from_sim no)
@@
 		(fields_autoplaced yes)
 		(property "Reference" "H1"
-			(at 49.53 170.1799 0)
+			(at 69.85 113.0299 0)
 			(effects
 				(font
@@
 		)
 		(property "Value" "MountingHole"
-			(at 49.53 172.7199 0)
+			(at 69.85 115.5699 0)
 			(effects
 				(font
@@
 		)
 		(property "Footprint" "MountingHole:MountingHole_3.2mm_M3"
-			(at 46.99 171.45 0)
+			(at 67.31 114.3 0)
 			(effects
 				(font
@@
 		)
 		(property "Datasheet" "~"
-			(at 46.99 171.45 0)
+			(at 67.31 114.3 0)
 			(effects
 				(font
@@
 		)
 		(property "Description" "Mounting Hole without connection"
-			(at 46.99 171.45 0)
+			(at 67.31 114.3 0)
 			(effects
 				(font
@@
 	(symbol
 		(lib_id "power:GND")
-		(at 39.37 104.14 0)
+		(at 77.47 95.25 0)
 		(unit 1)
 		(exclude_from_sim no)
@@
 		(fields_autoplaced yes)
 		(property "Reference" "#PWR07"
-			(at 39.37 110.49 0)
+			(at 77.47 101.6 0)
 			(effects
 				(font
@@
 		)
 		(property "Value" "GND"
-			(at 39.37 109.22 0)
+			(at 77.47 100.33 0)
 			(effects
 				(font
@@
 		)
 		(property "Footprint" ""
-			(at 39.37 104.14 0)
+			(at 77.47 95.25 0)
 			(effects
 				(font
@@
 		)
 		(property "Datasheet" ""
-			(at 39.37 104.14 0)
+			(at 77.47 95.25 0)
 			(effects
 				(font
@@
 		)
 		(property "Description" ""
-			(at 39.37 104.14 0)
+			(at 77.47 95.25 0)
 			(effects
 				(font
@@
 	(symbol
 		(lib_id "Connector:Conn_01x02_Socket")
-		(at 34.29 100.33 180)
+		(at 72.39 91.44 180)
 		(unit 1)
 		(exclude_from_sim no)
@@
 		(fields_autoplaced yes)
 		(property "Reference" "J1"
-			(at 34.925 92.71 0)
+			(at 73.025 83.82 0)
 			(effects
 				(font
@@
 		)
 		(property "Value" "Conn_01x02_Socket"
-			(at 34.925 95.25 0)
+			(at 73.025 86.36 0)
 			(effects
 				(font
@@
 		)
 		(property "Footprint" "TerminalBlock_Phoenix:TerminalBlock_Phoenix_MKDS-1,5-2_1x02_P5.00mm_Horizontal"
-			(at 34.29 100.33 0)
+			(at 72.39 91.44 0)
 			(effects
 				(font
@@
 		)
 		(property "Datasheet" "~"
-			(at 34.29 100.33 0)
+			(at 72.39 91.44 0)
 			(effects
 				(font
@@
 		)
 		(property "Description" ""
-			(at 34.29 100.33 0)
+			(at 72.39 91.44 0)
 			(effects
 				(font
@@
 		(fields_autoplaced yes)
 		(property "Reference" "Q2"
-			(at 128.27 100.33 0)
-			(effects
-				(font
-					(size 1.27 1.27)
-				)
-				(justify left)
-			)
-		)
-		(property "Value" "IPP50R280CE"
-			(at 128.27 102.87 0)
+			(at 128.27 100.3299 0)
+			(effects
+				(font
+					(size 1.27 1.27)
+				)
+				(justify left)
+			)
+		)
+		(property "Value" "IGLD60R190D1"
+			(at 128.27 102.8699 0)
 			(effects
 				(font
@@
 	(symbol
 		(lib_id "Mechanical:MountingHole")
-		(at 71.12 181.61 0)
+		(at 91.44 124.46 0)
 		(unit 1)
 		(exclude_from_sim no)
@@
 		(fields_autoplaced yes)
 		(property "Reference" "H4"
-			(at 73.66 180.3399 0)
+			(at 93.98 123.1899 0)
 			(effects
 				(font
@@
 		)
 		(property "Value" "MountingHole"
-			(at 73.66 182.8799 0)
+			(at 93.98 125.7299 0)
 			(effects
 				(font
@@
 		)
 		(property "Footprint" "MountingHole:MountingHole_3.2mm_M3"
-			(at 71.12 181.61 0)
+			(at 91.44 124.46 0)
 			(effects
 				(font
@@
 		)
 		(property "Datasheet" "~"
-			(at 71.12 181.61 0)
+			(at 91.44 124.46 0)
 			(effects
 				(font
@@
 		)
 		(property "Description" "Mounting Hole without connection"
-			(at 71.12 181.61 0)
+			(at 91.44 124.46 0)
 			(effects
 				(font
@@
 	(symbol
 		(lib_id "Mechanical:MountingHole")
-		(at 46.99 181.61 0)
+		(at 67.31 124.46 0)
 		(unit 1)
 		(exclude_from_sim no)
@@
 		(fields_autoplaced yes)
 		(property "Reference" "H3"
-			(at 49.53 180.3399 0)
+			(at 69.85 123.1899 0)
 			(effects
 				(font
@@
 		)
 		(property "Value" "MountingHole"
-			(at 49.53 182.8799 0)
+			(at 69.85 125.7299 0)
 			(effects
 				(font
@@
 		)
 		(property "Footprint" "MountingHole:MountingHole_3.2mm_M3"
-			(at 46.99 181.61 0)
+			(at 67.31 124.46 0)
 			(effects
 				(font
@@
 		)
 		(property "Datasheet" "~"
-			(at 46.99 181.61 0)
+			(at 67.31 124.46 0)
 			(effects
 				(font
@@
 		)
 		(property "Description" "Mounting Hole without connection"
-			(at 46.99 181.61 0)
-			(effects
-				(font
+			(at 67.31 124.46 0)
+			(effects
+				(font
